Commit message: Fully sync master with working code on laptop

File: frost-dev/example/minitaur Bound/urdf/minitaurWithTailFrontOffsetAccurate.urdf (robot description, URDF)
Before this commit: robot minitaur, 20 links, 19 joints
Links:
- added link tail_shaft, mass 0.107; collision cylinder length=0.05 radius=0.025; visual cylinder length=0.60 radius=0.01
- link tail_link: mass 0.4 -> 0.193
- link tail_mount: mass 0.9 -> 0.753; geometry collision box size=0.02 0.02 .02; visual box size=0.05 0.05 .05
- link tail_rotor: geometry collision cylinder length=0.55 radius=0.03; visual cylinder length=0.03 radius=0.05
Joints:
- added joint tail_shaft_joint: type fixed, parent tail_rotor, child tail_shaft, origin xyz=0 0 0 rpy=0 0 0
