Commit message: Add RML Template first draft, clear out a lot of junk

File: frost-dev/example/minitaur Bound/urdf/minitaurAccurate.urdf (robot description, URDF)
Before this commit: robot minitaur, 17 links, 16 joints
Joints:
- joint motor_back_leftL_joint: origin xyz=-0.225 0.13 0 rpy=0 0 3.14159 -> xyz=-0.2 0.125 0 rpy=0 0 3.14159
- joint motor_back_leftR_joint: origin xyz=-0.225 0.13 0 rpy=0 0 0 -> xyz=-0.2 0.125 0 rpy=0 0 0
- joint motor_back_rightL_joint: origin xyz=-0.225 -0.13 0 rpy=0 0 0 -> xyz=-0.2 -0.125 0 rpy=0 0 0
- joint motor_back_rightR_joint: origin xyz=-0.225 -0.13 0 rpy=0 0 3.14159 -> xyz=-0.2 -0.125 0 rpy=0 0 3.14159
- joint motor_front_leftL_joint: origin xyz=0.225 0.13 0 rpy=0 0 3.14159 -> xyz=0.2 0.125 0 rpy=0 0 3.14159
- joint motor_front_leftR_joint: origin xyz=0.225 0.13 0 rpy=0 0 0 -> xyz=0.2 0.125 0 rpy=0 0 0
- joint motor_front_rightL_joint: origin xyz=0.225 -0.13 0 rpy=0 0 0 -> xyz=0.2 -0.125 0 rpy=0 0 0
- joint motor_front_rightR_joint: origin xyz=0.225 -0.13 0 rpy=0 0 3.14159 -> xyz=0.2 -0.125 0 rpy=0 0 3.14159
