Commit message: update gaits, add min GRF constraint

File: frost-dev/example/minitaur Acceleration/urdf/minitaurWithTailBackOffsetAccurateG4.urdf (robot description, URDF)
Before this commit: robot minitaur, 21 links, 20 joints
Links:
- link tail_link: mass 0.033 -> 0.193
- link tail_shaft: mass 0.047 -> 0.107

File: frost-dev/example/minitaur Acceleration/urdf/minitaurWithTailBackOffsetAerodynamic.urdf (robot description, URDF)
Before this commit: robot minitaur, 21 links, 20 joints
Links:
- link tail_mount: mass 0.453 -> 0.634
- link tail_shaft: geometry collision cylinder length=0.05 radius=0.025; visual cylinder length=1.00 radius=0.01

File: frost-dev/example/minitaur Acceleration/urdf/minitaurWithTailBackOffsetAerodynamicG4.urdf (robot description, URDF)
Before this commit: robot minitaur, 21 links, 20 joints
Links:
- link tail_link: mass 0.033 -> 0.043
- link tail_shaft: mass 0.047 -> 0.057; geometry collision cylinder length=0.05 radius=0.025; visual cylinder length=1.00 radius=0.01
