Commit message: Update acceleration urdfs, gaits, and plotting

File: frost-dev/example/minitaur Acceleration/urdf/minitaurWithTailAccurateG4.urdf (robot description, URDF)
Before this commit: robot minitaur, 21 links, 20 joints
Links:
- link tail_link: mass 0.033 -> 0.193
- link tail_rotor: mass 0.0693 -> 0.0771
- link tail_shaft: mass 0.047 -> 0.107
Joints:
- joint tail_base_joint: origin xyz=-0.1 0 0.1 rpy=0 0 0 -> xyz=0 -0.1 0.1 rpy=0 0 0
- joint tail_joint: origin xyz=-0.1 0 0.1 rpy=0 0 0 -> xyz=0 0 0.1 rpy=0 0 0

File: frost-dev/example/minitaur Acceleration/urdf/minitaurWithTailAerodynamicG4.urdf (robot description, URDF)
Before this commit: robot minitaur, 21 links, 20 joints
Links:
- link tail_link: mass 0.033 -> 0.043
- link tail_rotor: mass 0.0693 -> 0.0771
- link tail_shaft: mass 0.047 -> 0.057; geometry collision cylinder length=0.05 radius=0.025; visual cylinder length=1.00 radius=0.01
Joints:
- joint tail_base_joint: origin xyz=-0.1 0 0.1 rpy=0 0 0 -> xyz=0 -0.1 0.1 rpy=0 0 0
- joint tail_joint: origin xyz=-0.1 0 0.1 rpy=0 0 0 -> xyz=0 0 0.1 rpy=0 0 0

File: frost-dev/example/minitaur Acceleration/urdf/minitaurWithTailAerodynamicRealisticG4.urdf (robot description, URDF)
Before this commit: robot minitaur, 21 links, 20 joints
Links:
- link tail_rotor: mass 0.0693 -> 0.0771
Joints:
- joint tail_base_joint: origin xyz=-0.1 0 0.1 rpy=0 0 0 -> xyz=0 -0.1 0.1 rpy=0 0 0
- joint tail_joint: origin xyz=-0.1 0 0.1 rpy=0 0 0 -> xyz=0 0 0.1 rpy=0 0 0

File: frost-dev/example/minitaur Acceleration/urdf/minitaurWithTailBackOffsetAccurateG4.urdf (robot description, URDF)
Before this commit: robot minitaur, 21 links, 20 joints
Joints:
- joint motor_back_leftL_joint: origin xyz=-0.225 0.13 0 rpy=0 0 3.14159 -> xyz=-0.2 0.125 0 rpy=0 0 3.14159
- joint motor_back_leftR_joint: origin xyz=-0.225 0.13 0 rpy=0 0 0 -> xyz=-0.2 0.125 0 rpy=0 0 0
- joint motor_back_rightL_joint: origin xyz=-0.225 -0.13 0 rpy=0 0 0 -> xyz=-0.2 -0.125 0 rpy=0 0 0
- joint motor_back_rightR_joint: origin xyz=-0.225 -0.13 0 rpy=0 0 3.14159 -> xyz=-0.2 -0.125 0 rpy=0 0 3.14159
- joint motor_front_leftL_joint: origin xyz=0.225 0.13 0 rpy=0 0 3.14159 -> xyz=0.2 0.125 0 rpy=0 0 3.14159
- joint motor_front_leftR_joint: origin xyz=0.225 0.13 0 rpy=0 0 0 -> xyz=0.2 0.125 0 rpy=0 0 0
- joint motor_front_rightL_joint: origin xyz=0.225 -0.13 0 rpy=0 0 0 -> xyz=0.2 -0.125 0 rpy=0 0 0
- joint motor_front_rightR_joint: origin xyz=0.225 -0.13 0 rpy=0 0 3.14159 -> xyz=0.2 -0.125 0 rpy=0 0 3.14159

File: frost-dev/example/minitaur Acceleration/urdf/minitaurWithTailBackOffsetAerodynamicG4.urdf (robot description, URDF)
Before this commit: robot minitaur, 21 links, 20 joints
Joints:
- joint motor_back_leftL_joint: origin xyz=-0.225 0.13 0 rpy=0 0 3.14159 -> xyz=-0.2 0.125 0 rpy=0 0 3.14159
- joint motor_back_leftR_joint: origin xyz=-0.225 0.13 0 rpy=0 0 0 -> xyz=-0.2 0.125 0 rpy=0 0 0
- joint motor_back_rightL_joint: origin xyz=-0.225 -0.13 0 rpy=0 0 0 -> xyz=-0.2 -0.125 0 rpy=0 0 0
- joint motor_back_rightR_joint: origin xyz=-0.225 -0.13 0 rpy=0 0 3.14159 -> xyz=-0.2 -0.125 0 rpy=0 0 3.14159
- joint motor_front_leftL_joint: origin xyz=0.225 0.13 0 rpy=0 0 3.14159 -> xyz=0.2 0.125 0 rpy=0 0 3.14159
- joint motor_front_leftR_joint: origin xyz=0.225 0.13 0 rpy=0 0 0 -> xyz=0.2 0.125 0 rpy=0 0 0
- joint motor_front_rightL_joint: origin xyz=0.225 -0.13 0 rpy=0 0 0 -> xyz=0.2 -0.125 0 rpy=0 0 0
- joint motor_front_rightR_joint: origin xyz=0.225 -0.13 0 rpy=0 0 3.14159 -> xyz=0.2 -0.125 0 rpy=0 0 3.14159

File: frost-dev/example/minitaur Deceleration/urdf/minitaurWithTailBackOffsetAerodynamicRealisticG4.urdf (robot description, URDF)
Before this commit: robot minitaur, 21 links, 20 joints
Joints:
- joint motor_back_leftL_joint: origin xyz=-0.225 0.13 0 rpy=0 0 3.14159 -> xyz=-0.2 0.125 0 rpy=0 0 3.14159
- joint motor_back_leftR_joint: origin xyz=-0.225 0.13 0 rpy=0 0 0 -> xyz=-0.2 0.125 0 rpy=0 0 0
- joint motor_back_rightL_joint: origin xyz=-0.225 -0.13 0 rpy=0 0 0 -> xyz=-0.2 -0.125 0 rpy=0 0 0
- joint motor_back_rightR_joint: origin xyz=-0.225 -0.13 0 rpy=0 0 3.14159 -> xyz=-0.2 -0.125 0 rpy=0 0 3.14159
- joint motor_front_leftL_joint: origin xyz=0.225 0.13 0 rpy=0 0 3.14159 -> xyz=0.2 0.125 0 rpy=0 0 3.14159
- joint motor_front_leftR_joint: origin xyz=0.225 0.13 0 rpy=0 0 0 -> xyz=0.2 0.125 0 rpy=0 0 0
- joint motor_front_rightL_joint: origin xyz=0.225 -0.13 0 rpy=0 0 0 -> xyz=0.2 -0.125 0 rpy=0 0 0
- joint motor_front_rightR_joint: origin xyz=0.225 -0.13 0 rpy=0 0 3.14159 -> xyz=0.2 -0.125 0 rpy=0 0 3.14159
