Commit message: Get basic simulation of Vision60 working, modified HybridSystem/simulate.m and calcDesiredStates

File: frost-dev/example/Planning Validation/urdf/vision60.urdf (robot description, URDF)
Before this commit: robot ngr, 17 links, 16 joints
Joints:
- joint 0: type revolute -> continuous
- joint 1: type revolute -> continuous
- joint 10: type revolute -> continuous
- joint 11: type revolute -> continuous
- joint 2: type revolute -> continuous
- joint 3: type revolute -> continuous
- joint 4: type revolute -> continuous
- joint 5: type revolute -> continuous
- joint 6: type revolute -> continuous
- joint 7: type revolute -> continuous
- joint 8: type revolute -> continuous
- joint 9: type revolute -> continuous
